Commit message: Updated some values

File: description/gazebo_control.xacro (robot description, xacro)
@@ -2,5 +2,5 @@
 <robot xmlns:xacro="http://www.ros.org/wiki/xacro">
    <gazebo>
-    <plugin name="gz::sim::systems:DiffDrive" filename="gz-sim-diff-drive-system">
+    <plugin name="gz::sim::systems::DiffDrive" filename="gz-sim-diff-drive-system">
         <!--wheel Information-->
         <left_joint>left_wheel_joint</left_joint>

File: description/robot_core.xacro (robot description, xacro)
@@ -23,5 +23,5 @@
 <link name="chassis">
     <visual>
-        <origin xyz="0.15 0 0.075" rpy="0 0 0"/>
+        <origin xyz="0.15 0 0.075"/>
         <geometry>
             <box size="0.3 0.3 0.15"/>
@@ -39,4 +39,7 @@
     </xacro:inertial_box>
 </link>
+<gazebo reference="chassis">
+  <material>Gazebo/White</material>
+</gazebo>
 <!-- LEFT WHEEL -->
 <joint name="left_wheel_joint" type="continuous">
@@ -58,8 +61,11 @@
         </geometry>
     </collision>
-    <xacro:inertial_cylinder mass="0.1" length="0.05" radius="0.05">
+    <xacro:inertial_cylinder mass="0.1" length="0.04" radius="0.05">
         <origin xyz="0 0 0" rpy="0 0 0"/>
     </xacro:inertial_cylinder>
 </link>
+<gazebo reference="left_wheel">
+  <material>Gazebo/Blue</material>
+</gazebo>
 <!-- RIGHT WHEEL -->
 <joint name="right_wheel_joint" type="continuous">
@@ -81,13 +87,16 @@
         </geometry>
     </collision>
-    <xacro:inertial_cylinder mass="0.1" length="0.05" radius="0.05">
+    <xacro:inertial_cylinder mass="0.1" length="0.04" radius="0.05">
         <origin xyz="0 0 0" rpy="0 0 0"/>
     </xacro:inertial_cylinder>
 </link>
+<gazebo reference="right_wheel">
+  <material>Gazebo/Blue</material>
+</gazebo>
 <!-- CASTER WHEEL -->
 <joint name="caster_wheel_joint" type="fixed">
     <parent link="chassis"/>
     <child link="caster_wheel"/>
-    <origin xyz="0.24 0 0" rpy="0 0 0"/>
+    <origin xyz="0.24 0 0"/>
 </joint>
 <link name="caster_wheel">
@@ -102,4 +111,9 @@
     </xacro:inertial_sphere>
 </link>
+<gazebo reference="caster_wheel">
+  <material>Gazebo/Black</material>
+  <mu1 value="0.001"/>
+  <mu2 value="0.001"/>
+</gazebo>
 </robot>
   <!-- Base Link

Commit message: update the gazebo_control xacro

File: description/gazebo_control.xacro (robot description, xacro)
@@ -6,6 +6,6 @@
         <left_joint>left_wheel_joint</left_joint>
         <right_joint>right_wheel_joint</right_joint>
-        <wheel_separation>0.14</wheel_separation>
-        <wheel_radius>0.02</wheel_radius>
+        <wheel_separation>0.297</wheel_separation>
+        <wheel_radius>0.05</wheel_radius>
         <!-- <<max_wheel_torque>200</max_wheel_torque>
          <max_wheel_acceleration>10.0</max_wheel_acceleration -->

File: description/robot_core.xacro (robot description, xacro)
@@ -23,5 +23,5 @@
 <link name="chassis">
     <visual>
-        <origin xyz="0.15 0 0.075"/>
+        <origin xyz="0.15 0 0.125"/>
         <geometry>
             <box size="0.3 0.3 0.15"/>
@@ -30,5 +30,5 @@
     </visual>
     <collision>
-        <origin xyz="0.15 0 0.075" rpy="0 0 0"/>
+        <origin xyz="0.15 0 0.125" rpy="0 0 0"/>
         <geometry>
             <box size="0.3 0.3 0.15"/>
@@ -36,5 +36,5 @@
     </collision>
     <xacro:inertial_box mass="0.5" x="0.3" y="0.3" z="0.15">
-        <origin xyz="0.15 0 0.075" rpy="0 0 0"/>
+        <origin xyz="0.15 0 0.125" rpy="0 0 0"/>
     </xacro:inertial_box>
 </link>
@@ -46,5 +46,5 @@
     <parent link="base_link"/>
     <child link="left_wheel"/>
-    <origin xyz="0 0.175 0" rpy="-${pi/2} 0 0"/>
+    <origin xyz="0 0.175 0.05" rpy="-${pi/2} 0 0"/>
     <axis xyz="0 0 1"/>
 </joint>
@@ -72,5 +72,5 @@
     <parent link="base_link"/>
     <child link="right_wheel"/>
-    <origin xyz="0 -0.175 0" rpy="${pi/2} 0 0"/>
+    <origin xyz="0 -0.175 0.05" rpy="${pi/2} 0 0"/>
     <axis xyz="0 0 -1"/>
 </joint>
@@ -98,5 +98,5 @@
     <parent link="chassis"/>
     <child link="caster_wheel"/>
-    <origin xyz="0.24 0 0"/>
+    <origin xyz="0.24 0 0.05"/>
 </joint>
 <link name="caster_wheel">
